File: hpcsadapter.sch (KiCad schematic (older format))
At the start: 20 parts, among them J1 Conn_01x08, J2 1761469-1, J3 73725-0110BLF, U1 TPS54327

Commit message: BOM completed
Parts:
- C1: DigiKey_PN (none) -> 311-1903-1-ND; Manufacturer (none) -> Yageo; Mfr_PN (none) -> CC0805MKX5R8BB226
- C2: DigiKey_PN (none) -> 311-1456-1-ND; Manufacturer (none) -> Yageo; Mfr_PN (none) -> CC0805KKX7R8BB105
- C3: DigiKey_PN (none) -> 311-1131-1-ND; Manufacturer (none) -> Yageo; Mfr_PN (none) -> CC0805KRX7R9BB332
- C4: DigiKey_PN (none) -> 311-1141-1-ND; Manufacturer (none) -> Yageo; Mfr_PN (none) -> CC0805KRX7R8BB104
- C5: DigiKey_PN (none) -> 311-1099-1-ND; Manufacturer (none) -> Yageo; Mfr_PN (none) -> CC0805JRNPO9BN100
- C6: DigiKey_PN (none) -> 587-5465-1-ND; Manufacturer (none) -> Taiyo Yuden; Mfr_PN (none) -> LMK212BBJ476MG-T
- J1: DigiKey_PN (none) -> ED2950-ND; Manufacturer (none) -> On Shore Technology Inc.; Mfr_PN (none) -> OSTYK42108030
- R1: DigiKey_PN (none) -> 311-22.0KCRCT-ND; Manufacturer (none) -> Yageo; Mfr_PN (none) -> RC0805FR-0722KL
- R2: DigiKey_PN (none) -> 311-10.2KCRCT-ND; Manufacturer (none) -> Yageo; Mfr_PN (none) -> RC0805FR-0710K2L
- R3: DigiKey_PN (none) -> 311-133KCRCT-ND; Manufacturer (none) -> Yageo; Mfr_PN (none) -> RC0805FR-07133KL
- R4: DigiKey_PN (none) -> 311-24.0KCRCT-ND; Manufacturer (none) -> Yageo; Mfr_PN (none) -> RC0805FR-0724KL
- R5, R7: DigiKey_PN (none) -> 311-43.0KCRCT-ND; Manufacturer (none) -> Yageo; Mfr_PN (none) -> RC0805FR-0743KL
- R6, R8: DigiKey_PN (none) -> 311-51.0KCRCT-ND; Manufacturer (none) -> Yageo; Mfr_PN (none) -> RC0805FR-0751KL

Commit message: separate out non-plated holes
Parts:
- C1: DigiKey_PN 311-1903-1-ND -> (none); MFR (none) -> Yageo; MPN (none) -> CC0805MKX5R8BB226; Manufacturer Yageo -> (none); Mfr_PN CC0805MKX5R8BB226 -> (none); SPN (none) -> 311-1903-1-ND; SPR (none) -> DigiKey
- C2: DigiKey_PN 311-1456-1-ND -> (none); MFR (none) -> Yageo; MPN (none) -> CC0805KKX7R8BB105; Manufacturer Yageo -> (none); Mfr_PN CC0805KKX7R8BB105 -> (none); SPN (none) -> 311-1456-1-ND; SPR (none) -> DigiKey
- C3: DigiKey_PN 311-1131-1-ND -> (none); MFR (none) -> Yageo; MPN (none) -> CC0805KRX7R9BB332; Manufacturer Yageo -> (none); Mfr_PN CC0805KRX7R9BB332 -> (none); SPN (none) -> 311-1131-1-ND; SPR (none) -> DigiKey
- C4: DigiKey_PN 311-1141-1-ND -> (none); MFR (none) -> Yageo; MPN (none) -> CC0805KRX7R8BB104; Manufacturer Yageo -> (none); Mfr_PN CC0805KRX7R8BB104 -> (none); SPN (none) -> 311-1141-1-ND; SPR (none) -> DigiKey
- C5: DigiKey_PN 311-1099-1-ND -> (none); MFR (none) -> Yageo; MPN (none) -> CC0805JRNPO9BN100; Manufacturer Yageo -> (none); Mfr_PN CC0805JRNPO9BN100 -> (none); SPN (none) -> 311-1099-1-ND; SPR (none) -> DigiKey
- C6: DigiKey_PN 587-5465-1-ND -> (none); MFR (none) -> Taiyo Yuden; MPN (none) -> LMK212BBJ476MG-T; Manufacturer Taiyo Yuden -> (none); Mfr_PN LMK212BBJ476MG-T -> (none); SPN (none) -> 587-5465-1-ND; SPR (none) -> DigiKey
- J1: value Conn_01x08 -> OSTYK42108030; DigiKey_PN ED2950-ND -> (none); MFR (none) -> On Shore Technology Inc.; MPN (none) -> OSTYK42108030; Manufacturer On Shore Technology Inc. -> (none); Mfr_PN OSTYK42108030 -> (none); SPN (none) -> ED2950-ND; SPR (none) -> DigiKey
- J2: DigiKey_PN 1761469-1-ND -> (none); MFR (none) -> TE; MPN (none) -> 1761469-1; Manufacturer TE -> (none); Mfr_PN 1761469-1 -> (none); SPN (none) -> 1761469-1-ND; SPR (none) -> DigiKey
- J3: DigiKey_PN 609-1041-ND -> (none); MFR (none) -> Amphenol FCI; MPN (none) -> 73725-0110BLF; Manufacturer Amphenol FCI -> (none); Mfr_PN 73725-0110BLF -> (none); SPN (none) -> 609-1041-ND; SPR (none) -> DigiKey
- L1: DigiKey_PN SDR0805-3R3MLCT-ND -> (none); MFR (none) -> Bourns; MPN (none) -> SDR0805-3R3ML; Manufacturer Bourns -> (none); Mfr_PN SDR0805-3R3ML -> (none); SPN (none) -> SDR0805-3R3MLCT-ND; SPR (none) -> DigiKey
- R1: DigiKey_PN 311-22.0KCRCT-ND -> (none); MFR (none) -> Yageo; MPN (none) -> RC0805FR-0722KL; Manufacturer Yageo -> (none); Mfr_PN RC0805FR-0722KL -> (none); SPN (none) -> 311-22.0KCRCT-ND; SPR (none) -> DigiKey
- R2: DigiKey_PN 311-10.2KCRCT-ND -> (none); MFR (none) -> Yageo; MPN (none) -> RC0805FR-0710K2L; Manufacturer Yageo -> (none); Mfr_PN RC0805FR-0710K2L -> (none); SPN (none) -> 311-10.2KCRCT-ND; SPR (none) -> DigiKey
- R3: DigiKey_PN 311-133KCRCT-ND -> (none); MFR (none) -> Yageo; MPN (none) -> RC0805FR-07133KL; Manufacturer Yageo -> (none); Mfr_PN RC0805FR-07133KL -> (none); SPN (none) -> 311-133KCRCT-ND; SPR (none) -> DigiKey
- R4: DigiKey_PN 311-24.0KCRCT-ND -> (none); MFR (none) -> Yageo; MPN (none) -> RC0805FR-0724KL; Manufacturer Yageo -> (none); Mfr_PN RC0805FR-0724KL -> (none); SPN (none) -> 311-24.0KCRCT-ND; SPR (none) -> DigiKey
- R5, R7: DigiKey_PN 311-43.0KCRCT-ND -> (none); MFR (none) -> Yageo; MPN (none) -> RC0805FR-0743KL; Manufacturer Yageo -> (none); Mfr_PN RC0805FR-0743KL -> (none); SPN (none) -> 311-43.0KCRCT-ND; SPR (none) -> DigiKey
- R6, R8: DigiKey_PN 311-51.0KCRCT-ND -> (none); MFR (none) -> Yageo; MPN (none) -> RC0805FR-0751KL; Manufacturer Yageo -> (none); Mfr_PN RC0805FR-0751KL -> (none); SPN (none) -> 311-51.0KCRCT-ND; SPR (none) -> DigiKey
- S1: DigiKey_PN EG2355-ND -> (none); MFR (none) -> E-Switch; MPN (none) -> 100SP1T1B4M2QE; Manufacturer E-Switch -> (none); Mfr_PN 100SP1T1B4M2QE -> (none); SPN (none) -> EG2355-ND; SPR (none) -> DigiKey
- U1: DigiKey_PN 296-28061-1-ND -> (none); MFR (none) -> Texas Instruments; MPN (none) -> TPS54327DDAR; Manufacturer Texas Instruments -> (none); Mfr_PN TPS54327DDAR -> (none); SPN (none) -> 296-28061-1-ND; SPR (none) -> DigiKey
